File: projects/pet-eletrica-ufc/boards/01-logic-gates/01-logic-gates.kicad_sch (KiCad schematic)
At the start: 18 parts, among them J1 5V INPUT, SW1 B3F-4050, SW2 B3F-4050, U1 SN74HC08N, U2 SN74HC32N, U3 SN74HC04N

Commit message: feat(pet-ufc): implement discrete transistor logic board
Parts:
- removed C2, C3: 100nF 50V, Capacitor_THT:C_Disc_D5.0mm_W2.5mm_P2.50mm, symbol Device:C
- removed U1: SN74HC08N, Package_DIP:DIP-14_W7.62mm, symbol PET_Logic:SN74HC08
- removed U2: SN74HC32N, Package_DIP:DIP-14_W7.62mm, symbol PET_Logic:SN74HC32
- removed U3: SN74HC04N, Package_DIP:DIP-14_W7.62mm, symbol PET_Logic:SN74HC04
- added Q1, Q10, Q2, Q3, Q4, Q5, Q6, Q7, Q8, Q9: 2N3904, Package_TO_SOT_THT:TO-92_Inline, symbol Transistor_BJT:Q_NPN_EBC
- added R10, R11, R12, R21, R22, R23, R6, R7, R8, R9: 10k 5%, Resistor_THT:R_Axial_DIN0207_L6.3mm_D2.5mm_P10.16mm_Horizontal, symbol Device:R
- added R13, R14, R15, R16, R17: 2.2k 5%, Resistor_THT:R_Axial_DIN0207_L6.3mm_D2.5mm_P10.16mm_Horizontal, symbol Device:R
- added R18, R19, R20: 1.5k 5%, Resistor_THT:R_Axial_DIN0207_L6.3mm_D2.5mm_P10.16mm_Horizontal, symbol Device:R
- added SW3, SW4, SW5: B3F-4050, Button_Switch_THT:SW_SPST_Omron_B3F-50xx, symbol Switch:SW_Push
- D1: value TLHR5200 -> 1N5819; footprint LED_THT:LED_D5.0mm -> Diode_THT:D_DO-41_SOD81_P10.16mm_Horizontal; symbol Device:LED -> Device:D_Schottky
- D4: value 1N5819 -> TLHR5200; footprint Diode_THT:D_DO-41_SOD81_P10.16mm_Horizontal -> LED_THT:LED_D5.0mm; symbol Device:D_Schottky -> Device:LED
- R3, R4, R5: value 1.5k 5% -> 10k 5%
Connections:
- net 5V_IN: now also D1.2 (A); no longer D4.2 (A)
- net GND: now also Q10.1 (E), Q2.1 (E), Q3.1 (E), Q4.1 (E), Q5.1 (E), Q6.1 (E), Q7.1 (E), Q8.1 (E), Q9.1 (E), R21.2, R22.2, R23.2; no longer D1.1 (K), D2.1 (K), D3.1 (K)
- net VCC: now also D1.1 (K), R13.1, R14.1, R15.1, R16.1, R17.1, R18.1, R19.1, R20.1, SW3.1, SW4.1, SW5.1; no longer D4.1 (K)
- net Y_AND: now also Q3.3 (C), R14.2, R6.1; no longer R3.1
- net Y_NOT: now also Q9.3 (C), R12.1, R17.2; no longer R5.1
- net Y_OR: now also Q7.3 (C), R10.1, R16.2; no longer R4.1
- net A renamed A_AND
- net A_AND: now also R3.1
- net B renamed B_AND
- net B_AND: now also R4.1
- net LED1_A renamed Q1_B
- net Q1_B: now also Q1.2 (B); no longer D1.2 (A)
- net LED2_A renamed LED_AND_A
- net LED_AND_A: now also R18.2; no longer R4.2
- net LED3_A renamed LED_OR_A
- net LED_OR_A: now also R19.2; no longer R5.2
- new net A_NOT: R11.1, R23.1, SW5.2
- new net A_OR: R21.1, R7.1, SW3.2
- new net B_OR: R22.1, R8.1, SW4.2
- new net LED_AND_K: D2.1 (K), Q4.3 (C)
- new net LED_NOT_A: D4.2 (A), R20.2
- new net LED_NOT_K: D4.1 (K), Q10.3 (C)
- new net LED_OR_K: D3.1 (K), Q8.3 (C)
- new net N_AND: Q1.3 (C), R13.2, R5.1
- new net N_AND_MID: Q1.1 (E), Q2.3 (C)
- new net N_OR: Q5.3 (C), Q6.3 (C), R15.2, R9.1
- new net Q10_B: Q10.2 (B), R12.2
- new net Q2_B: Q2.2 (B), R4.2
- new net Q3_B: Q3.2 (B), R5.2
- new net Q4_B: Q4.2 (B), R6.2
- new net Q5_B: Q5.2 (B), R7.2
- new net Q6_B: Q6.2 (B), R8.2
- new net Q7_B: Q7.2 (B), R9.2
- new net Q8_B: Q8.2 (B), R10.2
- new net Q9_B: Q9.2 (B), R11.2
- no-connect marks 11 -> 0
Other:
- note added: "AND: series NAND plus inverter and LED driver"
- note added: "NOT: common-emitter inverter and LED driver"
- note added: "OR: parallel NOR plus inverter and LED driver"
- moved on the sheet: C1, D2, D3, J1, R1, R2, R3, R4, R5, SW1, SW2
